Commit message: feat(vision): Add core modules - camera URDF, detector and data

File: openarm_description/urdf/robot/openarm_robot.xacro (robot description, xacro)
@@ -178,3 +178,29 @@
         </xacro:if>
   </xacro:macro>
+<link name="camera_link">
+    <visual>
+      <geometry>
+        <box size="0.05 0.03 0.03"/>
+      </geometry>
+      <material name="black">
+        <color rgba="0 0 0 1"/>
+      </material>
+    </visual>
+    <collision>
+      <geometry>
+        <box size="0.05 0.03 0.03"/>
+      </geometry>
+    </collision>
+  </link>
+  <joint name="camera_joint" type="fixed">
+    <parent link="base_link"/>
+    <child link="camera_link"/>
+    <origin xyz="0.5 0.0 0.8" rpy="0.0 1.57 0.0"/>
+  </joint>
+  <link name="camera_optical_frame"/>
+  <joint name="camera_optical_joint" type="fixed">
+    <parent link="camera_link"/>
+    <child link="camera_optical_frame"/>
+    <origin xyz="0 0 0" rpy="-1.57 0 -1.57"/>
+  </joint>
 </robot>

Commit message: feat(integration): Update Visual System (Camera URDF + Object Detector)

File: openarm_description/urdf/robot/openarm_robot.xacro (robot description, xacro)
@@ -178,3 +178,58 @@
         </xacro:if>
   </xacro:macro>
+<link name="camera_link">
+    <visual>
+      <geometry>
+        <box size="0.05 0.03 0.03"/>
+      </geometry>
+      <material name="black">
+        <color rgba="0 0 0 1"/>
+      </material>
+    </visual>
+    <collision>
+      <geometry>
+        <box size="0.05 0.03 0.03"/>
+      </geometry>
+    </collision>
+  </link>
+  <joint name="camera_joint" type="fixed">
+    <parent link="base_link"/>
+    <child link="camera_link"/>
+    <origin xyz="0.5 0.0 0.8" rpy="0.0 1.57 0.0"/>
+  </joint>
+  <link name="camera_optical_frame"/>
+  <joint name="camera_optical_joint" type="fixed">
+    <parent link="camera_link"/>
+    <child link="camera_optical_frame"/>
+    <origin xyz="0 0 0" rpy="-1.57 0 -1.57"/>
+  </joint>
+<gazebo reference="camera_link">
+    <sensor type="depth" name="depth_camera_sensor">
+      <always_on>true</always_on>
+      <update_rate>30.0</update_rate>
+      <camera name="camera">
+        <horizontal_fov>1.047</horizontal_fov> <image>
+          <width>640</width>
+          <height>480</height>
+          <format>R8G8B8</format>
+        </image>
+        <clip>
+          <near>0.05</near>
+          <far>8.0</far>
+        </clip>
+      </camera>
+      <plugin name="depth_camera_controller" filename="libgazebo_ros_camera.so">
+        <ros>
+          <namespace>openarm</namespace>
+          <remapping>custom_camera/image_raw:=/camera/image_raw</remapping>
+          <remapping>custom_camera/camera_info:=/camera/camera_info</remapping>
+          <remapping>custom_camera/points:=/camera/points</remapping>
+          <remapping>custom_camera/depth/image_raw:=/camera/depth/image_raw</remapping>
+        </ros>
+        <frame_name>camera_optical_frame</frame_name>
+        <min_depth>0.1</min_depth>
+        <max_depth>8.0</max_depth>
+      </plugin>
+    </sensor>
+  </gazebo>
 </robot>
